File: Heaterboard.brd (EAGLE design)
At the start: 138.2 x 29.1 mm, 35 parts, among them IC2 ATTINY10, J1 POWER_JACK, T1 2N3904, U1 2N3906, U2 LM35DT, U3 2N3906, U4 ULN2003A, U5 W25Q32FV

Commit message: corrected reversed LM35
Parts:
- moved U2 5.09 mm to (135.1, 16.3), turned to 0 degrees
Routing:
- net +5V: track 146.9 -> 139.8 mm
- net N$1: track 74.2 -> 78.0 mm
Changed lines of the file:
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@@
 <attribute name="VALUE" x="83.5415" y="27.1058" size="1.78045" layer="25" ratio="10" rot="R180"/>
 </element>
-<element name="U2" library="partlibrary" package="TA03F" value="LM35DT" x="130.048" y="16.002" smashed="yes" rot="R180">
-<attribute name="MANUFACTURER_PART_NUMBER" value="LM35DT" x="130.048" y="16.002" size="1.778" layer="27" rot="R180" display="off"/>
-<attribute name="NAME" x="131.5974" y="14.605" size="1.27" layer="25" ratio="6" rot="SR0"/>
-<attribute name="VENDOR" value="Texas Instruments" x="130.048" y="16.002" size="1.778" layer="27" rot="R180" display="off"/>
+<element name="U2" library="partlibrary" package="TA03F" value="LM35DT" x="135.128" y="16.256" smashed="yes">
+<attribute name="MANUFACTURER_PART_NUMBER" value="LM35DT" x="135.128" y="16.256" size="1.778" layer="27" display="off"/>
+<attribute name="NAME" x="133.5786" y="17.653" size="1.27" layer="25" ratio="6" rot="SR180"/>
+<attribute name="VENDOR" value="Texas Instruments" x="135.128" y="16.256" size="1.778" layer="27" display="off"/>
 </element>
 <element name="5V" library="testpad" library_urn="urn:adsk.eagle:library:385" package="P1-13" package3d_urn="urn:adsk.eagle:package:27946/1" value="PTR1PAD1-13" x="33.528" y="25.908" smashed="yes" rot="R180">
@@
 </polygon>
 <contactref element="C1" pad="1"/>
-<wire x1="135.128" y1="17.018" x2="134.9756" y2="17.1704" width="1.27" layer="16"/>
-<wire x1="134.9756" y1="17.1704" x2="134.9756" y2="18.30455625" width="1.27" layer="16"/>
-<wire x1="134.9756" y1="18.30455625" x2="133.21415625" y2="20.066" width="1.27" layer="16"/>
-<wire x1="133.21415625" y1="20.066" x2="127.508" y2="20.066" width="1.27" layer="16"/>
-<wire x1="121.92" y1="16.256" x2="123.698" y2="16.256" width="1.27" layer="16"/>
-<wire x1="123.698" y1="16.256" x2="125.73" y2="18.288" width="1.27" layer="16"/>
-<wire x1="125.73" y1="18.288" x2="127.508" y2="20.066" width="1.27" layer="16"/>
 <wire x1="121.92" y1="16.256" x2="115.57" y2="16.256" width="1.27" layer="16"/>
 <wire x1="107.95" y1="26.637" x2="105.123" y2="29.464" width="1.27" layer="16"/>
@@
 <contactref element="TIVA" pad="21"/>
 <contactref element="J1" pad="PWR"/>
-<wire x1="128.54" y1="5.842" x2="125.73" y2="8.652" width="1.27" layer="16"/>
-<wire x1="125.73" y1="8.652" x2="125.73" y2="18.288" width="1.27" layer="16"/>
+<wire x1="128.54" y1="5.842" x2="127.508" y2="6.874" width="1.27" layer="16"/>
+<wire x1="130.048" y1="15.24" x2="129.032" y2="16.256" width="1.27" layer="16"/>
+<wire x1="129.032" y1="16.256" x2="127.508" y2="16.256" width="1.27" layer="16"/>
+<wire x1="127.508" y1="16.256" x2="121.92" y2="16.256" width="1.27" layer="16"/>
+<wire x1="127.508" y1="20.066" x2="127.508" y2="16.256" width="1.27" layer="16"/>
+<wire x1="127.508" y1="16.256" x2="127.508" y2="6.874" width="1.27" layer="16"/>
+<wire x1="127.508" y1="25.146" x2="127.508" y2="27.686" width="0" layer="19" extent="1-1"/>
+<wire x1="127.508" y1="22.606" x2="127.508" y2="25.146" width="0" layer="19" extent="1-1"/>
+<wire x1="127.508" y1="20.066" x2="127.508" y2="22.606" width="0" layer="19" extent="1-1"/>
 </signal>
 <signal name="GND" class="2" airwireshidden="yes">
@@
 <wire x1="109.474" y1="16.002" x2="109.474" y2="13.462" width="0.254" layer="1"/>
 <wire x1="109.474" y1="13.462" x2="110.998" y2="11.938" width="0.254" layer="1"/>
-<wire x1="124.968" y1="11.938" x2="130.048" y2="17.018" width="0.254" layer="1"/>
-<wire x1="110.998" y1="11.938" x2="124.968" y2="11.938" width="0.254" layer="1"/>
+<wire x1="133.9050375" y1="14.0170375" x2="135.128" y2="15.24" width="0.254" layer="1"/>
+<wire x1="133.9050375" y1="14.0170375" x2="127.508" y2="11.938" width="0.254" layer="1"/>
+<wire x1="110.998" y1="11.938" x2="127.508" y2="11.938" width="0.254" layer="1"/>
 </signal>
 <signal name="N$3">
