File: Heaterboard.sch (EAGLE design)
At the start: 14 parts, among them IC1 EK-TM4C123GXLP, J1 POWER_JACK, U1 CSD18504KCS, U2 LM35DT

Commit message: checkpoint for schematic capture
Parts:
- removed JP1, JP2: (no value), pinhead:PINHD-2X10/90
- removed U$1, U$2: YSD-160AB3C-8, SparkFun-LED:7-SEGMENT-1DIGIT-1INCH-BLUE
- added LED1, LED2: LA-401AD, led-7-segment:LA-401AD
- added R2: (no value), resistor:R-US_R1206
- added R3: (no value), resistor:R-US_0207/10
- added U3: TLC5926IDBQRDBQ24-M, partlibrary:TLC5926IDBQRDBQ24-M
Connections:
- removed net N$2: IC1.PB5, JP1.3
- removed net N$21: IC1.PC5, JP2.9
- removed net N$22: IC1.PC6, JP2.11
- removed net N$23: IC1.PC7, JP2.13
- removed net N$24: IC1.PD6, JP2.15
- removed net N$25: IC1.PD7, JP2.17
- removed net N$26: IC1.PF4, JP2.19
- removed net N$27: IC1.PB2, JP2.4
- removed net N$28: IC1.PE0, JP2.6
- removed net N$29: IC1.PF0, JP2.8
- removed net N$3: IC1.PB0, JP1.5
- removed net N$30: IC1.RESET, JP2.10
- removed net N$31: IC1.PB7, JP2.12
- removed net N$32: IC1.PB6, JP2.14
- removed net N$33: IC1.PA4, JP2.16
- removed net N$34: IC1.PA3, JP2.18
- removed net N$35: IC1.PA2, JP2.20
- removed net N$4: IC1.PB1, JP1.7
- new net CLK: IC1.PD0, U3.CLK
- new net FSS: IC1.PD1
- new net LE: U3.LE(ED1)
- new net N$40: R2.1, R3.1, U3.R-EXT
- new net OE: U3.!OE(ED2)
- new net SDI: IC1.PD3, U3.SDI
- new net SDO: IC1.PD2, U3.SDO
- net +3V3: now also LED1.A@1, LED1.A@2, LED2.A@1, LED2.A@2; no longer JP1.1
- net +5V: now also U3.VDD; no longer JP1.2
- net GND: now also R2.2, R3.2, U3.GND; no longer JP1.4, JP2.2
- net N$10: now also LED1.F, U3.OUT5; no longer IC1.PA7, JP1.19
- net N$11: now also LED1.G, U3.OUT6; no longer IC1.PD0, JP1.6
- net N$12: now also LED1.DP, U3.OUT7; no longer IC1.PD1, JP1.8
- net N$13: now also LED2.DP, U3.OUT8; no longer IC1.PD2, JP1.10
- net N$14: now also LED2.G, U3.OUT9; no longer IC1.PD3, JP1.12
- net N$15: now also LED2.F, U3.OUT10; no longer IC1.PE2, JP1.16
- net N$16: now also LED2.E, U3.OUT11; no longer IC1.PF1, JP1.20
- net N$17: now also LED2.D, U3.OUT12; no longer IC1.PF2, JP2.1
- net N$18: now also LED2.C, U3.OUT13; no longer IC1.PF3, JP2.3
- net N$19: now also LED2.B, U3.OUT14; no longer IC1.PB3, JP2.5
- net N$20: now also LED2.A, U3.OUT15; no longer IC1.PC4, JP2.7
- net N$5: now also LED1.A, U3.OUT0; no longer IC1.PE4, JP1.9
- net N$6: now also LED1.B, U3.OUT1; no longer IC1.PE5, JP1.11
- net N$7: now also LED1.C, U3.OUT2; no longer IC1.PB4, JP1.13
- net N$8: now also LED1.D, U3.OUT3; no longer IC1.PA5, JP1.15
- net N$9: now also LED1.E, U3.OUT4; no longer IC1.PA6, JP1.17
- net PWR_ON: no longer JP1.14
- net T-SENSE: no longer JP1.18
Other:
- note added: "Note: this device is only upside down in the schematic"
- note added: "R2 and R3 represent the same resistor, and are to be considered mutually exclusive. R2 proides a SMT footprint, R3 provides a through-hole footprint."
- note added: "The TLC59 is connected via a SPI-like interface."
- note added: "The TLC5926 is basically a combination of shift register and LED driver. It is capable of sinking up to 120mA, configurable, at a wide range of voltages. It is designed to work with common-cathode LEDs."
- note added: "This resistor is massively overkill for this task. So is the NMOS. This design will probably require significant thermal mass."
- note added: "VSS and VDD are isolated from the TIVA board's power and ground, and are sourced through the power jack adjacent to the heater."
- moved on the sheet: J1, R1, TP1, TP2, U1

Commit message: checkpoint before massive rework
Connections:
- net N$1 renamed HEATER_ON
- removed net FSS: IC1.PD1
- net LE: now also IC1.PB7
- net OE: now also IC1.PB6
Other:
- note added: "The output is enabled and locked with a pair of dedicated GPIO"
- moved on the sheet: IC1, J1, R1, TP1, TP2, TP3, TP4, TP5, U1, U2

Commit message: final checkpoint
Parts:
- removed IC1: EK-TM4C123GXLP, EK-TM4C123GXL:EK-TM4C123GXLP
- removed LED1, LED2: LA-401AD, led-7-segment:LA-401AD
- removed R3: (no value), resistor:R-US_0207/10
- removed TP1, TP2, TP3, TP4, TP5: PTR1PAD1-13, testpad:PTR1PAD1-13
- added 3V, 5V, GND: PTR1PAD1-13, testpad:PTR1PAD1-13
- added 7SEG: NTE3074, partlibrary:NTE3074
- added C1: 10uF, resistor:C-US025-030X050
- added D2: (no value), adafruit:DIODEDO-1N4148
- added IC2: ATTINY10, adafruit:ATTINY10
- added JP1: (no value), pinhead:PINHD-1X10/90
- added JP2: (no value), pinhead:PINHD-1X2
- added JP4: (no value), pinhead:PINHD-1X8
- added LOGO1: OSHW-LOGOL, SparkFun-Aesthetics:OSHW-LOGOL
- added R10, R16: 330, resistor:R-US_0204/5
- added R11, R12, R13, R14, R15, R8, R9: 150, resistor:R-US_0204/5
- added R4, R5, R6, R7: 200, resistor:R-US_0207/10
- added T1: 2N3904, transistor:2N3904
- added TIP29: TIP29AG, partlibrary:TIP29AG
- added TIVA: EK-TM4C123GXLP, EK-TM4C123GXL:EK-TM4C123GXLP
- added U4: ULN2003A, partlibrary:ULN2003A
- added U5: W25Q32FV, SparkFun-IC-Memory:W25Q32FVSS
- R1: value PWR220T-20-50R0F -> 330; device partlibrary:PWR220T-20-50R0F -> resistor:R-US_0204/5
- R2: value (none) -> 10k; device resistor:R-US_R1206 -> resistor:R-US_0204/5
- U1: value CSD18504KCS -> 2N3906; device partlibrary:CSD18504KCS -> partlibrary:2N3906
- U3: value TLC5926IDBQRDBQ24-M -> 2N3906; device partlibrary:TLC5926IDBQRDBQ24-M -> partlibrary:2N3906
Connections:
- removed net HEATER_ON: R1.1, U1.DRAIN
- removed net LE: IC1.PB7, U3.LE(ED1)
- removed net N$11: LED1.G, U3.OUT6
- removed net N$18: LED2.C, U3.OUT13
- removed net N$40: R2.1, R3.1, U3.R-EXT
- removed net N$6: LED1.B, U3.OUT1
- removed net N$7: LED1.C, U3.OUT2
- removed net OE: IC1.PB6, U3.!OE(ED2)
- removed net PWR_ON: IC1.PE1, U1.GATE
- removed net SDI: IC1.PD3, U3.SDI
- removed net SDO: IC1.PD2, U3.SDO
- removed net VDD: J1.PWR, TP1.TP, U1.SOURCE
- removed net VSS: J1.GND, J1.GNDBREAK, R1.2, TP2.TP
- new net 1C: JP1.1, R8.2, U4.1C
- new net 2C: JP1.2, R9.2, U4.2C
- new net 3C: JP1.3, R15.2, U4.3C
- new net 4C: JP1.4, R12.2, U4.4C
- new net 5C: JP1.5, R11.2, U4.5C
- new net 6C: JP1.6, R14.2, U4.6C
- new net 7C: JP1.7, R13.2, U4.7C
- new net ANODE1: 7SEG.ANODE1, JP1.8, U1.C
- new net ANODE2: 7SEG.ANODE2, JP1.9, U3.C
- new net HEATER_COM: R4.1, R5.1, R6.1, R7.1, TIP29.C
- new net N$1: R2.1, U2.VOUT
- new net N$21: IC2.PB1, JP4.3, U5.!WP!(D2)
- new net N$23: IC2.VCC, JP4.5, U5.SI(D0)
- new net N$24: IC2./RST, JP4.6, U5.SCK
- new net N$25: JP4.7, U5.!HOLD!(D3)
- new net N$26: JP4.8, U5.VCC
- new net N$3: R16.1, T1.B
- new net N$4: T1.E, TIP29.B
- new net PA2: TIVA.PA2
- new net PA3: TIVA.PA3
- new net PA4: TIVA.PA4
- new net PA5: TIVA.PA5
- new net PA6: TIVA.PA6
- new net PB0: TIVA.PB0, U4.7B
- new net PB1: TIVA.PB1, U4.6B
- new net PB2: TIVA.PB2, U4.5B
- new net PB3: TIVA.PB3, U4.4B
- new net PB4: TIVA.PB4, U4.3B
- new net PB5: TIVA.PB5, U4.2B
- new net PB6: TIVA.PB6, U4.1B
- new net PB7: TIVA.PB7
- new net PC4: TIVA.PC4
- new net PC5: TIVA.PC5
- new net PC6: R1.1, TIVA.PC6
- new net PC7: R10.1, TIVA.PC7
- new net PD1: TIVA.PD1
- new net PD2: TIVA.PD2
- new net PD3: TIVA.PD3
- new net PD6: TIVA.PD6
- new net PD7: TIVA.PD7
- new net PE0: TIVA.PE0
- new net PE1: TIVA.PE1
- new net PE2: TIVA.PE2
- new net PE4: TIVA.PE4
- new net PE5: TIVA.PE5
- new net PF0: TIVA.PF0
- new net PF1: TIVA.PF1
- new net PF2: TIVA.PF2
- new net PF3: TIVA.PF3
- new net PF4: TIVA.PF4
- new net P_ON: R16.2, TIVA.PA7
- new net RESET: TIVA.RESET
- net +3V3: now also 3V.TP, D2.C, TIVA.+3.3V; no longer IC1.+3.3V, LED1.A@1, LED1.A@2, LED2.A@1, LED2.A@2, TP4.TP, U2.VS+
- net +5V: now also 5V.TP, C1.1, J1.PWR, R4.2, R5.2, R6.2, R7.2, T1.C, TIVA.+5V, U1.E, U2.VS+, U3.E; no longer IC1.+5V, TP3.TP, U3.VDD
- net CLK: now also TIVA.PD0; no longer IC1.PD0, U3.CLK
- net GND: now also C1.2, GND.TP, J1.GND, J1.GNDBREAK, JP1.10, JP2.1, JP2.2, TIP29.E, TIVA.GND, TIVA.GND2, U4.GND; no longer IC1.GND, IC1.GND2, R2.2, R3.2, TP5.TP, U3.GND
- net N$10: now also IC2.PB2, JP4.4, U5.GND; no longer LED1.F, U3.OUT5
- net N$12: now also 7SEG.B1, 7SEG.B2, R9.1; no longer LED1.DP, U3.OUT7
- net N$13: now also 7SEG.C1, 7SEG.C2, R15.1; no longer LED2.DP, U3.OUT8
- net N$14: now also 7SEG.D1, 7SEG.D2, R12.1; no longer LED2.G, U3.OUT9
- net N$15: now also 7SEG.E1, 7SEG.E2, R11.1; no longer LED2.F, U3.OUT10
- net N$16: now also 7SEG.F1, 7SEG.F2, R14.1; no longer LED2.E, U3.OUT11
- net N$17: now also 7SEG.G1, 7SEG.G2, R13.1; no longer LED2.D, U3.OUT12
- net N$19: now also IC2.PB0, JP4.1, U5.!CS!; no longer LED2.B, U3.OUT14
- net N$20: now also IC2.GND, JP4.2, U5.SO(D1); no longer LED2.A, U3.OUT15
- net N$5: now also R10.2, U1.B; no longer LED1.A, U3.OUT0
- net N$8: now also R1.2, U3.B; no longer LED1.D, U3.OUT3
- net N$9: now also 7SEG.A1, 7SEG.A2, R8.1; no longer LED1.E, U3.OUT4
- net T-SENSE: now also D2.A, R2.2, TIVA.PE3; no longer IC1.PE3, U2.VOUT
Other:
- note added: "Secret Programming Headers"
- note removed: "Note: this device is only upside down in the schematic"
- note removed: "R2 and R3 represent the same resistor, and are to be considered mutually exclusive. R2 proides a SMT footprint, R3 provides a through-hole footprint."
- note removed: "The TLC59 is connected via a SPI-like interface."
- note removed: "The TLC5926 is basically a combination of shift register and LED driver. It is capable of sinking up to 120mA, configurable, at a wide range of voltages. It is designed to work with common-cathode LEDs."
- note removed: "The output is enabled and locked with a pair of dedicated GPIO"
- note removed: "This resistor is massively overkill for this task. So is the NMOS. This design will probably require significant thermal mass."
- note removed: "VSS and VDD are isolated from the TIVA board's power and ground, and are sourced through the power jack adjacent to the heater."
- moved on the sheet: J1, R2, U2
